File: past revisions/KMB-20/KMB-20.sch (EAGLE design)
At the start: 140 parts, among them J1 503182-1852, J2 10118194-0001LF, J3 DCJ0303, Q1 IRLML2803, Q10 IRLML5103, Q11 IRLML5103, Q12 IRLML5103, Q13 IRLML5103, Q14 IRLML2803, Q15 IRLML2803, Q16 IRLML5103, Q2 IRLML2803, Q5 IRLML2803, Q6 IRLML2803, Q7 IRLML2803, Q8 IRLML2803, Q9 IRLML5103, U1 MAX706R, U12 EP2W+, U13 RFM23BP, U14 S1216V8, U15 XTB_2018_07_15, U16 XTB_2018_07_15, U17 XTB_2018_07_15, U18 XTB_2018_07_15, U2 FXAS21002FXAS21002, U20 MR25H40MDF, U3 LSM9DS1, U4 ATSAMD21G-A, U5 MAX4372TEUK+T, U6 LTC4121-4.2, U7 TPS54226PWPRPWP14_2P31X2P46-L, U8 PE014006, U9 PE014006, X1 BU-SMA-V, X2 BU-SMA-V, X3 BU-SMA-V, Y1 32.768kHz

Commit message: added KMB-22 design
Parts:
- removed 3.3V, GND: (no value), pinhead:PINHD-1X1
- removed FRAME5: FRAME-LETTER, SparkFun-Aesthetics:FRAME-LETTER
- removed J3: DCJ0303, maholli:DCJ0303
- removed Q10, Q11, Q12, Q13, Q16, Q9: IRLML5103, User-Submitted:MOSFET-PCHANNEL
- removed Q14, Q15, Q6, Q7, Q8: IRLML2803, maholli:IRLML2803TRPBF
- removed U12: EP2W+, maholli:EP2W+
- removed U13: RFM23BP, RFM23BP:RFM23BP
- removed U14: S1216V8, maholli:S1216V8
- removed U15, U16, U17, U18: XTB_2018_07_15, maholli:XTB_2018_07_15
- removed U20: MR25H40MDF, maholli:MR25H40MDF
- added C29, C30, C31, C32: .1uF, SparkFun-Capacitors:CAP0603-CAP
- added C33: 2.2uF, SparkFun-Capacitors:2.2UF-0603-10V-20%
- added JP19, JP20, JP21: JUMPER-PAD-3-2OF3_NC_BY_TRACE_SMALL, SparkFun-Passives:JUMPER-PAD-3-2OF3_NC_BY_TRACE_SMALL
- added JP22, JP28: (no value), pinhead:PINHD-1X1
- added Q3, Q4: IRLML5103, User-Submitted:MOSFET-PCHANNEL
- added R38, R39, R40, R41, R42: (no value), SparkFun-Resistors:RESISTOR0603
- added R43: 330, SparkFun-Resistors:330OHM1/10W1%(0603)
- added R44: 10K, SparkFun-Resistors:10KOHM-1/10W-1%(0603)0603
- added T1, T2, T3, T4, T5: NDS352A, zetex:PMOSSOT23
- added U10: EP2W+, maholli:EP2W+
- added U11: S1216V8, maholli:S1216V8
- C14: value 0.1uF -> 22uF; device SparkFun-Capacitors:0.1UF-25V(+80/-20%)(0603) -> SparkFun-Capacitors:22UF-0805-6.3V-20%
- C16: value 22uF -> 10uF; device SparkFun-Capacitors:22UF-0805-6.3V-20% -> SparkFun-Capacitors:10UF-0603-6.3V-20%
- C18: value 10uF -> 1.0uF; device SparkFun-Capacitors:10UF-0603-6.3V-20% -> SparkFun-Capacitors:1.0UF-0603-16V-10%
- C19: value 2.2uF -> 10uF; device SparkFun-Capacitors:2.2UF-0603-10V-20% -> SparkFun-Capacitors:10UF-0603-6.3V-20%
- C20: value 2.2nF -> 2.2uF; device SparkFun-Capacitors:2.2NF/2200PF-0603-50V-10% -> SparkFun-Capacitors:2.2UF-0603-10V-20%
- C21: value 10uF -> 2.2nF; device SparkFun-Capacitors:10UF-0603-6.3V-20% -> SparkFun-Capacitors:2.2NF/2200PF-0603-50V-10%
- C22: value 0.1uF -> .1uF; device SparkFun-Capacitors:1.0UF-0603-16V-10% -> SparkFun-Capacitors:CAP0603-CAP
- C23: value .1uF -> 0.1uF; device SparkFun-Capacitors:CAP0603-CAP -> SparkFun-Capacitors:0.1UF-0603-25V-5%
- C24: value 22uF -> 3.3nF; device SparkFun-Capacitors:0.1UF-0603-25V-5% -> SparkFun-Capacitors:3.3NF-0603-100V-10%
- C25: value 3.3nF -> 1.0uF; device SparkFun-Capacitors:3.3NF-0603-100V-10% -> SparkFun-Capacitors:1.0UF-0603-16V-10%
- C26: value 1.0uF -> 22uF; device SparkFun-Capacitors:1.0UF-0603-16V-10% -> SparkFun-Capacitors:0.1UF-0603-25V-5%
- C27: value 2.2uF -> 0.1uF; device SparkFun-Capacitors:2.2UF-0603-10V-20% -> SparkFun-Capacitors:0.1UF-0603-25V-5%
- C28: device SparkFun-Capacitors:0.1UF-25V(+80/-20%)(0603) -> SparkFun-Capacitors:0.1UF-0603-25V-5%
- J1: value 503182-1852 -> 1981584-1; device maholli:503182-1852 -> audio amplifier example:1981584-1
- J2: value 10118194-0001LF -> POWER_JACKPTH_LOCK; device 10118194-0001LF:10118194-0001LF -> SparkFun-Connectors:POWER_JACKPTH_LOCK
- JP10, JP13: value M023.5MM_LOCK -> (none); device SparkFun-Connectors:M023.5MM_LOCK -> SparkFun-Connectors:M03POLAR_LOCK
- JP15: value (none) -> M023.5MM_LOCK; device SparkFun-Connectors:M03POLAR_LOCK -> SparkFun-Connectors:M023.5MM_LOCK
- JP18: value JUMPER-PAD-3-2OF3_NC_BY_TRACE_SMALL -> M023.5MM_LOCK; device SparkFun-Passives:JUMPER-PAD-3-2OF3_NC_BY_TRACE_SMALL -> SparkFun-Connectors:M023.5MM_LOCK
- JP24: value JUMPER-PAD-3-2OF3_NC_BY_TRACE_SMALL -> (none); device SparkFun-Passives:JUMPER-PAD-3-2OF3_NC_BY_TRACE_SMALL -> pinhead:PINHD-1X1
- JP3: value JUMPER-PAD-3-2OF3_NC_BY_TRACE_SMALL -> (none); device SparkFun-Passives:JUMPER-PAD-3-2OF3_NC_BY_TRACE_SMALL -> pinhead:PINHD-1X2
- JP4: value JUMPER-PAD-3-2OF3_NC_BY_TRACE_SMALL -> (none); device SparkFun-Passives:JUMPER-PAD-3-2OF3_NC_BY_TRACE_SMALL -> pinhead:PINHD-1X3
- JP5: device SparkFun-Connectors:M03POLAR_LOCK -> pinhead:PINHD-1X6
- JP8: device SparkFun-Connectors:M03POLAR_LOCK -> pinhead:PINHD-1X3
- Q1, Q2, Q5: value IRLML2803 -> IRLML5103; device maholli:IRLML2803TRPBF -> User-Submitted:MOSFET-PCHANNEL
- R13: value 470k -> 22.1
- R14: value 22.1k -> 100K
- R15: value 4.7k -> 470k
- R16: value 6.04K -> 4.7k
- R17: value 100K -> 6.04K
- R18: value 10K -> 4.7K
- R19: value 4.7K -> 680
- R20: value 3.3K -> 10K
- R21: value 10k -> 3.3K; device SparkFun-Resistors:RESISTOR0603 -> resistor:R-US_R0603
- R22: value 10k -> 1k; device SparkFun-Resistors:RESISTOR0603 -> resistor:R-US_R0603
- R23, R24: value 10k -> 4; device SparkFun-Resistors:RESISTOR0603 -> resistor:R-US_R0603
- R25, R28, R37: value 4.7k -> (none)
- R26, R27: value 4.7k -> 4; device SparkFun-Resistors:RESISTOR0603 -> resistor:R-US_R0603
- R29, R30, R32: value 100k -> 4; device SparkFun-Resistors:RESISTOR0603 -> resistor:R-US_R0603
- R31, R7: value 100k -> (none)
- R33: value 330 -> 4; device SparkFun-Resistors:330OHM1/10W1%(0603) -> resistor:R-US_R0603
- R34: value 10K -> (none); device SparkFun-Resistors:10KOHM-1/10W-1%(0603)0603 -> SparkFun-Resistors:RESISTOR0603
- R35: value 0.025 -> (none); device resistor:R-US_R2512 -> SparkFun-Resistors:RESISTOR0603
- R36: value 10k -> (none)
- R4: value 10k -> 110K
- R5: value 110K -> 316K
- R6: value 316K -> (none); device SparkFun-Resistors:10KOHM-1/10W-1%(0603)0603 -> SparkFun-Resistors:RESISTOR0603
- U1: value MAX706R -> RFM23BP; device maholli:MAX708RESA-T -> RFM23BP:RFM23BP; SPICEPREFIX (none) -> U
- U2: value FXAS21002FXAS21002 -> LSM9DS1; device maholli:FXAS21002FXAS21002 -> SparkFun-Sensors:LSM9DS1
- U3: value LSM9DS1 -> MAX708RESA-T; device SparkFun-Sensors:LSM9DS1 -> maholli:MAX708RESA-T
- U6: value LTC4121-4.2 -> MAX4372TEUK+T; device BrownSpaceEngineering:LTC4121-4.2 -> maholli:MAX4372TEUK+T
- U8: value PE014006 -> LTC4121-4.2; device maholli:PE014005 -> BrownSpaceEngineering:LTC4121-4.2
- U9: value PE014006 -> LC05111C13MTTTG; device maholli:PE014005 -> BrownSpaceEngineering:LC05111C13MTTTG
Connections:
- removed net BURN_RELAY_A: Q2.G, U4.PA15(XOUT/SER2:3+)
- removed net BURN_RELAY_B: Q1.G, U4.PA18(SER1:2+)
- removed net ENAB_BURN5: R36.1, R37.2, U4.PA10(AIN18/SER0:2+)
- removed net GPS_PWR_IN: Q16.D, R34.2, U14.VCC, U14.V_BCKP
- removed net N$20: F2.1, J2.VDD
- removed net N$30: Q7.G, R27.1
- removed net N$39: R4.2, U4.PA06(AIN6/SER0:2/TC1:0)
- removed net N$43: J3.2, J3.3, JP10.2, JP11.2, JP12.1
- removed net N$53: D2.C, U4.PA08(I2C/AIN16/SER0:0+)
- removed net N$56: Q13.G, Q14.D, R7.1
- removed net N$57: Q14.G, R37.1
- removed net SPI_CS_MRAM: U20.!CS, U4.PB23(SER5:3+)
- removed net SPI_CS_RFM: U13.NSEL, U4.PB03(AIN11/SER5:1)
- removed net SPI_CS_SD: J1.CD/DAT3, U4.PA20(SER5:2+)
- removed net SPI_CS_XTB1: U15.SPI_CS, U4.PA28
- removed net SPI_CS_XTB2: U16.SPI_CS, U4.PB22(SER5:2+)
- removed net SPI_CS_XTB3: U17.SPI_CS, U4.PA16(I2C/SER1:0+)
- removed net SPI_CS_XTB4: U18.SPI_CS, U4.PA19(SER1:3+)
- removed net USB_D+: J2.D+, U4.PA25(SER3:3+)
- removed net USB_D-: J2.D-, U4.PA24(SER3:2+)
- removed net VBATT_IN: C27.1, F2.2, JP10.1, JP11.1, JP13.2
- removed net VBURN5: JP7.3, Q13.D
- removed net VBURN_A_IN: Q12.S, Q9.S, R31.2, R32.2, U9.11
- removed net VBURN_B_IN: Q10.S, Q11.S, Q13.S, R29.2, R30.2, R7.2, U8.11
- removed net WDT_WDI: U1.WDI, U4.PA17(I2C/SER1:1+)
- removed net XTB_RESET: U15.RESET, U16.RESET, U17.RESET, U18.RESET, U4.PA27
- new net DAC_0: JP22.1, U4.PA02(AIN0/DAC)
- new net GPS_1PPS: U11.1PPS, U4.PA03(AIN1/REFA)
- new net GPS_PWR: Q1.S, U11.VCC
- new net I_SOLAR: U4.PA08(I2C/AIN16/SER0:0+), U6.OUT
- new net LED_GRN: D2.C, U4.PB08(AIN2/SER4:0/TC4:0)
- new net N$41: C27.1, R19.1, U9.VCC
- new net N$42: C17.1, U7.VCC
- new net N$45: R22.2, U9.CS
- new net N_ENAB_REG: U4.PA16(I2C/SER1:0+), U7.EN
- new net PA04: U4.PA04(AIN4/REFB/SER0:0/TC0:0)
- new net PA12: JP24.1, U4.PA12(I2C/SER2:0+)
- new net PA15: U4.PA15(XOUT/SER2:3+)
- new net PB02: JP28.1, U4.PB02(AIN10/SER5:0)
- new net PB09: JP27.1, U4.PB09(AIN3/SER4:1/TC4:1)
- new net PB10: JP26.1, U4.PB10(SER4:2+)
- new net PB11: JP25.1, U4.PB11(SER4:3+)
- new net PB13: U4.PA13(I2C/SER2:1+)
- new net PWR_GND: C14.1, C15.1, C16.2, C17.2, C24.2, C25.2, R13.1, U7.EPAD, U7.GND, U7.PGND1, U7.PGND2
- new net SPI_SS: U1.NSEL, U4.PA28
- new net USB_D_N: J1.D-, U4.PA24(SER3:2+)
- new net USB_D_P: J1.D+, U4.PA25(SER3:3+)
- new net USB_ID: J1.ID, JP8.2
- new net VBURN_IN: Q2.D, Q3.D, Q4.D, Q5.D, R23.1, R24.1, R26.1, R27.1, R29.1, R30.1, R32.1, R33.1, R39.2, R40.2, R41.2, R42.2
- new net WDT_!PFO: U3.!PFO, U4.PA20(SER5:2+)
- new net WDT_!RESET: JP4.1, U3.!RESET
- new net WDT_PFI: U3.PFI, U4.PB22(SER5:2+)
- new net WDT_RESET: JP4.3, U3.RESET
- net !RESET: now also JP4.2, JP5.3; no longer JP27.1, U1.!RESET, U1.!WDO
- net 3.3V: now also C14.2, C22.1, JP20.3, JP21.3, JP3.2, JP5.2, JP8.1, Q1.D, R16.2, R21.1, R23.2, R24.2, R26.2, R27.2, R29.2, R30.2, R32.2, R43.2, R44.2, R7.1, U1.VCC, U11.V_BCKP, U6.RS-, U6.VCC; no longer 3.3V.1, C13.1, C16.2, J1.VDD, JP18.3, JP3.3, JP4.3, Q16.S, R13.2, R20.1, U13.VCC, U15.AVDD, U15.VDD(3.3V), U16.AVDD, U16.VDD(3.3V), U17.AVDD, U17.VDD(3.3V), U18.AVDD, U18.VDD(3.3V), U2.CS, U20.VDD, U3.VDD, U3.VDDIO
- net ENAB_BURN1: now also R35.1, U4.PB23(SER5:3+); no longer R24.1, U4.PB02(AIN10/SER5:0)
- net ENAB_BURN2: now also R36.1; no longer R23.1
- net ENAB_BURN3: now also R31.2, R37.1, U4.PA06(AIN6/SER0:2/TC1:0); no longer R22.1, R27.2, U4.PA09(I2C/AIN17/SER0:1+)
- net ENAB_BURN4: now also R34.2, R38.1, U4.PA07(AIN7/SER0:3/TC1:1); no longer R21.1, R26.2, U4.PA11(AIN19/SER0:3+)
- net ENAB_GPS: now also R20.2, U4.PA27; no longer R19.1, U4.PA07(AIN7/SER0:3/TC1:1)
- net GND: now also C20.2, C22.2, C28.2, C29.2, C30.2, C31.2, C32.2, C33.2, J1.GND, J1.S1, JP10.1, JP13.1, JP15.2, JP19.1, JP20.1, JP21.1, JP5.6, JP8.3, R17.1, R22.1, R25.1, R28.1, R31.1, R34.1, R4.1, T1.S, T2.S, T3.S, T4.S, T5.S, U1.GND1, U1.GND2, U1.GND3, U10.GND, U10.GND@1, U10.GND@10, U10.GND@11, U10.GND@12, U10.GND@13, U10.GND@14, U10.GND@16, U10.GND@17, U10.GND@18, U10.GND@19, U10.GND@2, U10.GND@20, U10.GND@21, U10.GND@22, U10.GND@23, U10.GND@24, U10.GND@25, U10.GND@27, U10.GND@28, U10.GND@29, U10.GND@3, U10.GND@30, U10.GND@31, U10.GND@32, U10.GND@5, U10.GND@6, U10.GND@7, U10.GND@8, U10.GND@9, U11.GND@10, U11.GND@12, U11.GND@13, U11.GND@24, U2.RES, U8.FREQ, U8.GND, U8.NC, U8.NTC, U9.S2, U9.TST, U9.VSS; no longer C14.2, C15.1, C16.1, C17.2, C18.2, C21.2, C24.2, C25.2, C28.1, GND.1, J1.SHIELD, J1.VSS, J2.GND, JP12.2, JP15.1, JP18.1, JP24.1, JP3.1, JP4.1, JP8.1, Q14.S, Q15.S, Q5.S, Q6.S, Q7.S, Q8.S, R14.1, R16.1, R21.2, R22.2, R23.2, R24.2, R36.2, R5.1, U1.GND, U1.PFI, U12.GND, U13.GND, U14.GND@10, U14.GND@12, U14.GND@13, U14.GND@24, U15.GND, U15.START, U16.GND, U16.START, U17.GND, U17.START, U18.GND, U18.START, U2.I2C/SPI, U20.EP, U20.VSS, U3.RES, U6.FREQ, U6.NC, U6.NTC, U7.EPAD, U7.GND, U7.PGND1, U7.PGND2, U8.12, U8.A2, U9.12, U9.A2
- net I2C_SCL: now also R2.1, U11.SCL/NC, U2.SCL/SPC, U4.PA10(AIN18/SER0:2+); no longer R3.1, U2.SCL/SCK, U3.SCL/SPC, U4.PA13(I2C/SER2:1+)
- net I2C_SDA: now also R3.1, U11.SDA/NC, U2.SDA/SDI/SDO, U4.PA09(I2C/AIN17/SER0:1+); no longer R2.1, U2.SDA/MOSI, U3.SDA/SDI/SDO, U4.PA12(I2C/SER2:0+)
- net I2C_SDOA/G: now also JP1.2, U2.SDO_A/G; no longer JP2.2, U3.SDO_A/G
- net I_BATT: now also U4.PA05(AIN5/SER0:1/TC0:1); no longer U4.PA04(AIN4/REFB/SER0:0/TC0:0)
- net L1_CHG: now also U8.RUN; no longer U6.RUN
- net L1_FAULTN: now also R16.1, U8.~FAULT; no longer R15.1, U6.~FAULT
- net L1_PROG: now also R17.2, U8.PROG; no longer R16.2, R4.1, U6.PROG
- net LION1: now also C26.1, R19.2, U8.BAT, U8.BATSNS; no longer C24.1, U6.BAT, U6.BATSNS
- net N$1: now also R43.1; no longer R33.1
- net N$10: now also C28.1, R20.1, T1.G; no longer Q15.G, R19.2
- net N$11: now also C31.1, R37.2, T4.G; no longer Q5.G, R25.1
- net N$12: now also Q1.G, R21.2, T1.D; no longer Q15.D, Q16.G, R20.2
- net N$13: now also F2.1, J1.VBUS; no longer C14.1, R5.2, R6.1, U4.PA05(AIN5/SER0:1/TC0:1)
- net N$14: now also C18.2; no longer C22.2
- net N$15: now also Q3.G, R40.1, T3.D; no longer Q12.G, Q8.D, R31.1
- net N$16: now also U10.PORT1; no longer U12.PORT1
- net N$17: now also U10.PORT2, X3.1; no longer U12.PORT2, X1.1
- net N$19: now also U1.ANT, X1.1; no longer U13.ANT, X3.1
- net N$2: now also U2.CAP; no longer U3.CAP
- net N$21: now also JP2.2, U2.SDO_M; no longer JP1.2, U3.SDO_M
- net N$22: now also J2.GND, J2.GNDBREAK, JP11.2, JP12.2, JP15.1; no longer C28.2, U2.VREGD
- net N$23: now also JP20.2, U2.CS_M; no longer JP3.2, U3.CS_M
- net N$24: now also JP19.3, R44.1; no longer JP24.3, R34.1
- net N$25: now also C29.1, R35.2, T2.G; no longer Q8.G, R28.1
- net N$26: now also JP21.2, U2.CS_A/G; no longer JP4.2, U3.CS_A/G
- net N$3: now also C18.1; no longer C22.1
- net N$32: now also C21.2, U8.SW; no longer C20.2, U6.SW
- net N$33: now also C21.1, U8.BOOST; no longer C20.1, U6.BOOST
- net N$34: now also C20.1, U8.INTVCC; no longer C19.1, U6.INTVCC
- net N$35: now also U8.MPPT; no longer U6.MPPT
- net N$36: now also U8.CHGSNS; no longer U6.CHGSNS
- net N$37: now also R15.1, U8.~CHRG; no longer R13.1, U6.~CHRG
- net N$38: now also C32.1, R38.2, T5.G; no longer Q2.S, U9.A1
- net N$4: now also JP16.1, JP18.2; no longer JP13.1, JP16.2
- net N$40: now also C13.1, R4.2, R5.1, U4.PA11(AIN19/SER0:3+); no longer Q1.S, U8.A1
- net N$44: now also Q4.G, R41.1, T4.D; no longer Q11.G, Q7.D, R30.1
- net N$46: now also C25.1, R14.2; no longer C26.1, R17.2
- net N$47: now also Q5.G, R42.1, T5.D; no longer Q10.G, Q6.D, R29.1
- net N$5: now also C30.1, R36.2, T3.G; no longer Q6.G, R26.1
- net N$51: now also C24.1; no longer C25.1
- net N$52: now also R13.2; no longer R14.2
- net N$6: now also U2.C1; no longer U3.C1
- net N$7: now also Q2.G, R39.1, T2.D; no longer Q5.D, Q9.G, R32.1
- net N$8: now also JP3.1, U3.VCC; no longer JP18.2, U1.VCC
- net N$9: now also JP19.2, U11.RSTN; no longer JP24.2, U14.RSTN
- net PGOOD: now also R14.1; no longer R17.1
- net RF_IN: now also U10.SUM_PORT, U11.RF_IN; no longer U12.SUM_PORT, U14.RF_IN
- net RF_NIRQ: now also U1.NIRQ, U4.PB03(AIN11/SER5:1); no longer U13.NIRQ, U4.PA02(AIN0/DAC)
- net RF_SDN: now also U1.SDN, U4.PA19(SER1:3+); no longer U13.SDN, U4.PA03(AIN1/REFA)
- net SPI_MISO: now also U1.SDO, U4.PA22(I2C/SER3:0+); no longer J1.DAT0, U13.SDO, U15.SPI_MISO, U16.SPI_MISO, U17.SPI_MISO, U18.SPI_MISO, U20.SO, U4.PA21(SER5:3+)
- net SPI_MOSI: now also U1.SDI, U4.PA21(SER5:3+); no longer J1.CMD, U13.SDI, U15.SPI_MOSI, U16.SPI_MOSI, U17.SPI_MOSI, U18.SPI_MOSI, U20.SI, U4.PA22(I2C/SER3:0+)
- net SPI_SCK: now also U1.SCK; no longer J1.CLK, U13.SCK, U15.SPI_SCK, U16.SPI_SCK, U17.SPI_SCK, U18.SPI_SCK, U20.SCK
- net SWCLK: now also JP5.4; no longer JP26.1
- net SWDIO: now also JP5.5; no longer JP25.1
- net UART1_RX: now also U11.TXD, U4.PA18(SER1:2+); no longer U14.TXD, U4.PB08(AIN2/SER4:0/TC4:0)
- net UART1_TX: now also U11.RXD, U4.PA17(I2C/SER1:1+); no longer U14.RXD, U4.PB09(AIN3/SER4:1/TC4:1)
- net VBATT: now also C33.1, F2.2, J2.PWR, JP11.1, JP12.1, JP16.2, JP18.1, R5.2; no longer J3.1, JP16.1, Q1.D, Q2.D, R35.2, U7.EN, U8.14, U9.14
- net VBURN1: now also Q2.S; no longer Q9.D
- net VBURN2: now also JP7.3, Q3.S; no longer JP5.3, Q12.D
- net VBURN3: now also JP10.3, Q4.S; no longer JP9.3, Q11.D
- net VBURN4: now also JP9.3, Q5.S; no longer JP8.3, Q10.D
- net VREG_IN: now also C16.1, R6.1; no longer C18.1, C21.1, R35.1, U7.VCC
- net VSOLAR: now also JP10.2, JP13.2, R7.2, U6.RS+; no longer JP15.2, JP5.2, JP8.2, JP9.2
- net VSOLAR_IN: now also C19.1, U8.IN; no longer C17.1, U6.IN
Other:
- note added: "4"
- note added: "ATSAMD21G18 32-bit ARM Microprocessor VDD Range: 1.62-3.63V"
- note added: "Buck Converter - 3.3V OUT"
- note added: "Burn Wire 1"
- note added: "Burn Wire 2"
- note added: "Burn Wire 3"
- note added: "Burn Wire 4"
- note added: "Burn Wire Control"
- note added: "FREQ tied to GND to select 750kHz switching frequency"
- note added: "LTC4121 can handle several amps of inrush current upon battery connection"
- note added: "NC tied to ground prevent charge buildup, approved by LT."
- note added: "NTC tied to GND b/c no NTC sensor"
- note added: "Place L1 near SW pin"
- note added: "R28 & R29 set Vmp=9V"
- note added: "RF Splitter - 2 Way, 0deg DC-Pass"
- note added: "Run pulled up to ensure charging on startup"
- note added: "Solar Panel Current Sensor"
- note added: "Spare IO breakout"
- note added: "To Do: XLab Mez board design Stretch Goals: Ultracap Power Supply Max GFET sensor"
- note added: "Ven threshold is 2.45V. Resistor divider sets RUN high when Solar Panel Voltage is >=6V."
- note removed: "3-AXIS GYROSCOPE"
- note removed: "5"
- note removed: "ADDRESS = 0x21"
- note removed: "ATSAMD21G18 32-bit ARM Microprocessor"
- note removed: "Antenna Board Connectors"
- note removed: "Burn Wire Control (Antenna Depolyment)"
- note removed: "Burn Wire Control (Sprite deployment)"
- note removed: "Decide on HOLD and !WP"
- note removed: "MRAM - Nonvolatile Memory (4MB storage)"
- note removed: "MicroSD Card"
- note removed: "PROG monitors charge current using: Ichrg=988*Vprog/Rprog"
- note removed: "Power Relay A"
- note removed: "Power Relay B"
- note removed: "RF Splitter (2 Way, 0deg DC-Pass)"
- note removed: "Regulator - 3.3V OUT"
- note removed: "Sensor Modules"
- note removed: "Solar Panel Board Connectors"
- note removed: "To Do: Characterize power consumption Validate SPI pinout of SAMD21"
- note removed: "VBATT 4.5 to 18V"
