File: past revisions/KMB-21/KMB-21.sch (EAGLE design)
At the start: 140 parts, among them J1 503182-1852, J2 10118194-0001LF, J3 DCJ0303, Q1 IRLML2803, Q10 IRLML5103, Q11 IRLML5103, Q12 IRLML5103, Q13 IRLML5103, Q14 IRLML2803, Q15 IRLML2803, Q16 IRLML5103, Q2 IRLML2803, Q5 IRLML2803, Q6 IRLML2803, Q7 IRLML2803, Q8 IRLML2803, Q9 IRLML5103, U1 MAX706R, U12 EP2W+, U13 RFM23BP, U14 S1216V8, U15 XTB_2018_07_15, U16 XTB_2018_07_15, U17 XTB_2018_07_15, U18 XTB_2018_07_15, U2 FXAS21002FXAS21002, U20 MR25H40MDF, U3 LSM9DS1, U4 ATSAMD21G-A, U5 MAX4372TEUK+T, U6 LTC4121-4.2, U7 TPS54226PWPRPWP14_2P31X2P46-L, U8 PE014006, U9 PE014006, X1 BU-SMA-V, X2 BU-SMA-V, X3 BU-SMA-V, Y1 32.768kHz

Commit message: added KMB-22 design
Parts:
- removed C28: 0.1uF, SparkFun-Capacitors:0.1UF-25V(+80/-20%)(0603)
- removed FRAME5: FRAME-LETTER, SparkFun-Aesthetics:FRAME-LETTER
- removed GND: (no value), pinhead:PINHD-1X1
- removed JP18: JUMPER-PAD-3-2OF3_NC_BY_TRACE_SMALL, SparkFun-Passives:JUMPER-PAD-3-2OF3_NC_BY_TRACE_SMALL
- removed JP7: (no value), SparkFun-Connectors:M03POLAR_LOCK
- removed Q13: IRLML5103, User-Submitted:MOSFET-PCHANNEL
- removed Q14: IRLML2803, maholli:IRLML2803TRPBF
- removed R36: 10k, SparkFun-Resistors:RESISTOR0603
- removed R37: 4.7k, SparkFun-Resistors:RESISTOR0603
- removed R7: 100k, SparkFun-Resistors:RESISTOR0603
- removed U15, U16, U17, U18: XTB_2018_07_15, maholli:XTB_2018_07_15
- removed U20: MR25H40MDF, maholli:MR25H40MDF
- added U10, U11: XTB_2018_04_25, maholli:XTB_2018_04_25
- U2: value FXAS21002FXAS21002 -> MR25H40; device maholli:FXAS21002FXAS21002 -> maholli:MR25H40
- renumbered Q15 to Q3, Q16 to Q4
Connections:
- removed net ENAB_BURN5: R36.1, R37.2, U4.PA10(AIN18/SER0:2+)
- removed net N$56: Q13.G, Q14.D, R7.1
- removed net N$57: Q14.G, R37.1
- removed net SPI_CS_XTB3: U17.SPI_CS, U4.PA16(I2C/SER1:0+)
- removed net SPI_CS_XTB4: U18.SPI_CS, U4.PA19(SER1:3+)
- removed net VBURN5: JP7.3, Q13.D
- new net GPS_1PPS: U14.1PPS, U4.PB08(AIN2/SER4:0/TC4:0)
- new net LED_1: D2.C, U4.PA07(AIN7/SER0:3/TC1:1)
- new net N$31: U2.!WP
- new net N$49: U2.!HOLD
- new net N$54: U4.PA16(I2C/SER1:0+)
- new net N$55: U4.PB10(SER4:2+)
- new net WDT_PWR: U1.VCC
- new net XTB_START: U10.START, U11.START, U4.PB02(AIN10/SER5:0)
- net !RESET: no longer U1.!WDO
- net 3.3V: now also U10.AVDD, U10.DVDD, U10.HALL_PWR, U10.INA_VDD, U11.AVDD, U11.DVDD, U11.HALL_PWR, U11.INA_VDD; no longer JP18.3, U15.AVDD, U15.VDD(3.3V), U16.AVDD, U16.VDD(3.3V), U17.AVDD, U17.VDD(3.3V), U18.AVDD, U18.VDD(3.3V), U2.CS, U2.VDD, U2.VDDIO, U20.VDD
- net BURN_RELAY_B: now also U4.PA10(AIN18/SER0:2+); no longer U4.PA18(SER1:2+)
- net ENAB_BURN1: now also U4.PB03(AIN11/SER5:1); no longer U4.PB02(AIN10/SER5:0)
- net ENAB_BURN4: now also U4.PA08(I2C/AIN16/SER0:0+); no longer U4.PA11(AIN19/SER0:3+)
- net ENAB_GPS: now also U4.PA06(AIN6/SER0:2/TC1:0); no longer U4.PA07(AIN7/SER0:3/TC1:1)
- net GND: now also U10.GND, U11.GND, U2.VSS; no longer C28.1, GND.1, JP18.1, JP7.1, Q14.S, R36.2, U1.PFI, U15.GND, U15.START, U16.GND, U16.START, U17.GND, U17.START, U18.GND, U18.START, U2.GND, U2.I2C/SPI, U20.EP, U20.VSS
- net I2C_SCL: no longer U2.SCL/SCK
- net I2C_SDA: no longer U2.SDA/MOSI
- net I_BATT: now also U4.PA05(AIN5/SER0:1/TC0:1); no longer U4.PA04(AIN4/REFB/SER0:0/TC0:0)
- net N$13: now also U4.PA11(AIN19/SER0:3+); no longer U4.PA05(AIN5/SER0:1/TC0:1)
- net N$22: now also U4.PA04(AIN4/REFB/SER0:0/TC0:0); no longer C28.2, U2.VREGD
- net N$39: now also U2.VDD; no longer R4.2, U4.PA06(AIN6/SER0:2/TC1:0)
- net N$53: now also U4.PA20(SER5:2+); no longer D2.C, U4.PA08(I2C/AIN16/SER0:0+)
- net N$8: now also R4.2, U4.PB11(SER4:3+); no longer JP18.2, U1.VCC
- net SPI_CS_MRAM: now also U2.!CI; no longer U20.!CS, U4.PB23(SER5:3+)
- net SPI_CS_RFM: now also U4.PA28; no longer U4.PB03(AIN11/SER5:1)
- net SPI_CS_SD: now also U4.PB23(SER5:3+); no longer U4.PA20(SER5:2+)
- net SPI_CS_XTB1: now also U10.SPI_CS, U4.PA27; no longer U15.SPI_CS, U4.PA28
- net SPI_CS_XTB2: now also U11.SPI_CS, U4.PB09(AIN3/SER4:1/TC4:1); no longer U16.SPI_CS, U4.PB22(SER5:2+)
- net SPI_MISO: now also U10.SPI_MISO, U11.SPI_MISO, U2.SO, U4.PA22(I2C/SER3:0+); no longer U15.SPI_MISO, U16.SPI_MISO, U17.SPI_MISO, U18.SPI_MISO, U20.SO, U4.PA21(SER5:3+)
- net SPI_MOSI: now also U10.SPI_MOSI, U11.SPI_MOSI, U2.SI, U4.PA21(SER5:3+); no longer U15.SPI_MOSI, U16.SPI_MOSI, U17.SPI_MOSI, U18.SPI_MOSI, U20.SI, U4.PA22(I2C/SER3:0+)
- net SPI_SCK: now also U10.SPI_SCK, U11.SPI_SCK, U2.SCK; no longer U15.SPI_SCK, U16.SPI_SCK, U17.SPI_SCK, U18.SPI_SCK, U20.SCK
- net UART1_RX: now also U4.PA18(SER1:2+); no longer U4.PB08(AIN2/SER4:0/TC4:0)
- net UART1_TX: now also U4.PA17(I2C/SER1:1+); no longer U4.PB09(AIN3/SER4:1/TC4:1)
- net VBURN_B_IN: no longer Q13.S, R7.2
- net VSOLAR: no longer JP7.2, JP8.2
- net WDT_WDI: now also U4.PA19(SER1:3+); no longer U4.PA17(I2C/SER1:1+)
- net XTB_RESET: now also U10.RESET, U11.RESET, U4.PB22(SER5:2+); no longer U15.RESET, U16.RESET, U17.RESET, U18.RESET, U4.PA27
Other:
- note added: "Antenna"
- note added: "Burn Wire Control"
- note added: "Power Relays"
- note added: "Spare IO breakout"
- note added: "Sprite deployment"
- note added: "Xlab Test Boards (XTB)"
- note removed: "3-AXIS GYROSCOPE"
- note removed: "ADDRESS = 0x21"
- note removed: "Antenna Board Connectors"
- note removed: "Burn Wire Control (Antenna Depolyment)"
- note removed: "Burn Wire Control (Sprite deployment)"
- note removed: "PROG monitors charge current using: Ichrg=988*Vprog/Rprog"
- note removed: "Power Relay A"
- note removed: "Power Relay B"
- note removed: "Sensor Modules"
- note removed: "Solar Panel Board Connectors"
