File: KMB-24.brd (EAGLE design)
At the start: 90.2 x 95.9 mm, 146 parts, among them J1 503182-1852, J2 10118194-0001LF, J3 DCJ0303, Q1 BC846, Q10 IRLML5103, Q11 IRLML5103, Q12 IRLML5103, Q13 IRLML5103, Q14 IRLML2803, Q15 IRLML2803, Q16 IRLML5103, Q2 BC846, Q5 IRLML2803, Q6 IRLML2803, Q7 IRLML2803, Q8 IRLML2803, Q9 IRLML5103, U1 MAX706R, U12 EP2W+, U13 RFM23BP, U14 S1216V8, U15 XTB_2018_07_15, U16 XTB_2018_07_15, U17 XTB_2018_07_15, U18 XTB_2018_07_15, U2 FXAS21002FXAS21002, U20 MR25H40MDF, U3 LSM9DS1, U4 ATSAMD21G-A, U5 MAX4372TEUK+T, U6 LTC4121-4.2, U7 TPS54226PWPRPWP14_2P31X2P46-L, U8 PE014006, U9 PE014006, X1 BU-SMA-V, X2 BU-SMA-V, X3 BU-SMA-V, Y1 32.768kHz

Commit message: added KMB-24
Parts:
- added D3, D4: SBR2A40P1Q-7, BrownSpaceEngineering:PWRDI-123
- Q1, Q2: value BC846 -> 2N5088
- moved R39 6.42 mm to (65.8, 72.2), turned to 180 degrees
- moved C27 2.79 mm to (65.7, 70.1)
- moved Q2 2.45 mm to (66.7, 74.8), turned to 90 degrees
- moved Q1 1.13 mm to (77.4, 37.4)
- moved R38 1.13 mm to (73.6, 37.3)
- moved R12 0.22 mm to (61.3, 78.1)
- moved R14 0.18 mm to (57.9, 78.1)
Connections:
- removed net GND4: R39.2
- removed net N$40: Q1.2, U8.1
- new net N$58: D4.A, Q1.3, U8.5
- net GND: now also Q1.2, Q2.2, R39.2; no longer U8.5, U9.5
- net N$38: now also D3.A, Q2.3, U9.5; no longer Q2.2, U9.1
- net VBATT: now also D3.C, D4.C, U8.1, U9.1; no longer Q1.3, Q2.3
Routing:
- net VBATT: track 152.0 -> 168.6 mm, vias 6 -> 5
- net N$58: track 0.00 -> 11.1 mm
- net N$38: track 11.1 -> 20.5 mm, vias 0 -> 1
- net BURN_RELAY_A: track 39.1 -> 32.9 mm
- net N$40: track 3.69 -> 0.00 mm
- net BURN_RELAY_B: track 35.3 -> 33.9 mm
- net GND4: track 1.09 -> 0.00 mm, vias 1 -> 0
- net GND: track 208.8 -> 209.5 mm, vias 140 -> 143
