File: KMB-24.sch (EAGLE design)
At the start: 145 parts, among them J1 503182-1852, J2 10118194-0001LF, J3 DCJ0303, Q1 BC846, Q10 IRLML5103, Q11 IRLML5103, Q12 IRLML5103, Q13 IRLML5103, Q14 IRLML2803, Q15 IRLML2803, Q16 IRLML5103, Q2 BC846, Q5 IRLML2803, Q6 IRLML2803, Q7 IRLML2803, Q8 IRLML2803, Q9 IRLML5103, U1 MAX706R, U12 EP2W+, U13 RFM23BP, U14 S1216V8, U15 XTB_2018_07_15, U16 XTB_2018_07_15, U17 XTB_2018_07_15, U18 XTB_2018_07_15, U2 FXAS21002FXAS21002, U20 MR25H40MDF, U3 LSM9DS1, U4 ATSAMD21G-A, U5 MAX4372TEUK+T, U6 LTC4121-4.2, U7 TPS54226PWPRPWP14_2P31X2P46-L, U8 PE014006, U9 PE014006, X1 BU-SMA-V, X2 BU-SMA-V, X3 BU-SMA-V, Y1 32.768kHz

Commit message: added KMB-24
Parts:
- added D3, D4: SBR2A40P1Q-7, BrownSpaceEngineering:DFLS130L
- Q1, Q2: value BC846 -> 2N5088
Connections:
- removed net GND4: R39.2
- removed net N$40: Q1.E, U8.A1
- new net N$58: D4.A, Q1.C, U8.A2
- net GND: now also Q1.E, Q2.E, R39.2; no longer U8.A2, U9.A2
- net N$38: now also D3.A, Q2.C, U9.A2; no longer Q2.E, U9.A1
- net VBATT: now also D3.C, D4.C, U8.A1, U9.A1; no longer Q1.C, Q2.C
Other:
- moved on the sheet: Q1, Q2, R38, R39
